File: eagle_design_files/V3/mk312lite_V3.brd (EAGLE design)
At the start: 90 x 120 mm, 101 parts, among them Q1 IRLL2705P, Q2 IRLL2705P, Q3 BSP170PH6327, Q4 IRLL2705P, Q5 IRLL2705P, Q6 BSP170PH6327, Q7 MMBT3904, Q8 MMBT3904, U1 ATMEGA16A, U10 LM358D, U3 4066D, U8B LTC1661, Y1 8MHZ

Commit message: Add files via upload
Parts:
- removed JP_5V: +5V, jumper:JP1
- removed JP_9V: +9V, jumper:JP1
Connections:
- net +5V: no longer JP_5V.1
- net +9V: no longer JP_9V.1
- net GND: no longer JP_5V.2, JP_9V.2
Routing:
- net +9V: track 262.4 -> 244.0 mm
- net +5V: track 626.9 -> 625.7 mm
Changed lines of the file:
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@@
 <attribute name="NAME" x="4.445" y="61.722" size="1.27" layer="25"/>
-</element>
-<element name="JP_5V" library="jumper" package="JP1" value="+5V" x="5.08" y="38.1" smashed="yes" rot="R270">
-<attribute name="NAME" x="2.794" y="40.132" size="1.27" layer="25" ratio="10"/>
-<attribute name="VALUE" x="2.54" y="35.179" size="1.27" layer="27" ratio="10"/>
-</element>
-<element name="JP_9V" library="jumper" package="JP1" value="+9V" x="12.7" y="38.1" smashed="yes" rot="R90">
-<attribute name="NAME" x="15.24" y="41.529" size="1.27" layer="25" ratio="10" rot="R180"/>
-<attribute name="VALUE" x="15.24" y="41.021" size="1.27" layer="27" ratio="10" rot="R180"/>
 </element>
 <element name="LCD1" library="MK312parts" package="LCD1602" package3d_urn="urn:adsk.eagle:package:6240760/1" value="HD44780LCD-1602" x="5.08" y="78.74" smashed="yes"/>
@@
 <contactref element="C9" pad="2"/>
 <contactref element="C11" pad="2"/>
-<contactref element="JP_5V" pad="2"/>
-<contactref element="JP_9V" pad="2"/>
 <contactref element="D1" pad="A"/>
 <contactref element="C10" pad="2"/>
@@
 <signal name="+5V" class="2">
 <contactref element="C10" pad="1"/>
-<contactref element="JP_5V" pad="1"/>
 <contactref element="U1" pad="29"/>
 <contactref element="U1" pad="27"/>
@@
 <wire x1="34.29" y1="2.54" x2="63.5" y2="2.54" width="0.635" layer="16"/>
 <wire x1="40.32" y1="13.65" x2="36.703" y2="10.033" width="0.635" layer="16"/>
-<wire x1="3.81" y1="38.1" x2="2.54" y2="38.1" width="0.635" layer="16"/>
 <wire x1="2.54" y1="3.81" x2="3.81" y2="2.54" width="0.635" layer="16"/>
 <wire x1="3.81" y1="2.54" x2="34.29" y2="2.54" width="0.635" layer="16"/>
@@
 </signal>
 <signal name="+9V" class="2">
-<contactref element="JP_9V" pad="1"/>
 <contactref element="C40" pad="2"/>
 <contactref element="C2" pad="+"/>
@@
 <wire x1="78.613" y1="52.07" x2="84.328" y2="46.355" width="1.27" layer="16"/>
 <wire x1="81.28" y1="23.79" x2="81.28" y2="27.94" width="1.27" layer="16"/>
-<wire x1="13.97" y1="38.1" x2="13.97" y2="25.4" width="0.508" layer="16"/>
-<wire x1="15.58" y1="23.79" x2="19.05" y2="23.79" width="0.508" layer="16"/>
-<wire x1="13.97" y1="25.4" x2="15.58" y2="23.79" width="0.508" layer="16"/>
 <wire x1="18.796" y1="23.241" x2="18.796" y2="23.622" width="0.3048" layer="16"/>
 <wire x1="18.796" y1="23.622" x2="19.05" y2="23.79" width="0.3048" layer="16"/>
