File: eagle_design_files/V3/mk312lite_V3.sch (EAGLE design)
At the start: 101 parts, among them Q1 IRLL2705P, Q2 IRLL2705P, Q3 BSP170PH6327, Q4 IRLL2705P, Q5 IRLL2705P, Q6 BSP170PH6327, Q7 MMBT3904, Q8 MMBT3904, U1 ATMEGA16A, U10 LM358D, U3 4066D, U8B LTC1661, Y1 8MHZ

Commit message: Add files via upload
Parts:
- removed JP_5V: +5V, jumper:JP1E
- removed JP_9V: +9V, jumper:JP1E
Connections:
- net +5V: no longer JP_5V.1
- net +9V: no longer JP_9V.1
- net GND: no longer JP_5V.2, JP_9V.2
Changed lines of the file:
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@@
 <part name="C41" library="rcl" library_urn="urn:adsk.eagle:library:334" deviceset="C-EU" device="C0805" package3d_urn="urn:adsk.eagle:package:23617/2" value="0.1uF"/>
 <part name="GND24" library="supply2" deviceset="GND" device=""/>
-<part name="JP_5V" library="jumper" deviceset="JP1E" device="" value="+5V"/>
-<part name="P+17" library="supply1" deviceset="+5V" device=""/>
-<part name="GND95" library="supply2" deviceset="GND" device=""/>
-<part name="JP_9V" library="jumper" deviceset="JP1E" device="" value="+9V"/>
-<part name="GND96" library="supply2" deviceset="GND" device=""/>
 <part name="U8B" library="MK312parts" deviceset="LTC1661IMS8" device="" value="LTC1661"/>
 <part name="P+4" library="supply1" library_urn="urn:adsk.eagle:library:371" deviceset="+5V" device=""/>
@@
 <part name="C5" library="rcl" library_urn="urn:adsk.eagle:library:334" deviceset="C-EU" device="C0805" package3d_urn="urn:adsk.eagle:package:23617/2" value="100pF"/>
 <part name="C7" library="rcl" library_urn="urn:adsk.eagle:library:334" deviceset="C-EU" device="C0805" package3d_urn="urn:adsk.eagle:package:23617/2" value="100pF"/>
-<part name="SUPPLY11" library="supply2" library_urn="urn:adsk.eagle:library:372" deviceset="+9V" device=""/>
 <part name="BAT" library="Rembrandt Electronics - JST XH Connectors v1-0" deviceset="JST-XH-02-PIN" device="-LONG-PAD" value="B2B-XH-A-GU"/>
 <part name="C10" library="rcl" library_urn="urn:adsk.eagle:library:334" deviceset="C-EU" device="C1206" package3d_urn="urn:adsk.eagle:package:23618/2" value="22uF"/>
@@
 <attribute name="VALUE" x="203.835" y="113.665" size="1.778" layer="96"/>
 </instance>
-<instance part="JP_5V" gate="A" x="129.54" y="78.74" smashed="yes" rot="R270">
-<attribute name="NAME" x="129.54" y="80.01" size="1.778" layer="95"/>
-<attribute name="VALUE" x="129.54" y="73.025" size="1.778" layer="96"/>
-</instance>
-<instance part="P+17" gate="1" x="119.38" y="78.74" smashed="yes" rot="MR270">
-<attribute name="VALUE" x="124.46" y="81.28" size="1.778" layer="96" rot="MR0"/>
-</instance>
-<instance part="GND95" gate="GND" x="124.46" y="71.12" smashed="yes">
-<attribute name="VALUE" x="122.555" y="67.945" size="1.778" layer="96"/>
-</instance>
-<instance part="JP_9V" gate="A" x="99.06" y="78.74" smashed="yes" rot="R270">
-<attribute name="NAME" x="99.06" y="80.01" size="1.778" layer="95"/>
-<attribute name="VALUE" x="99.06" y="73.025" size="1.778" layer="96"/>
-</instance>
-<instance part="GND96" gate="GND" x="93.98" y="71.12" smashed="yes">
-<attribute name="VALUE" x="92.075" y="67.945" size="1.778" layer="96"/>
-</instance>
 <instance part="D1" gate="G$1" x="149.86" y="114.3" smashed="yes" rot="R90">
 <attribute name="NAME" x="149.3774" y="116.84" size="1.778" layer="95" rot="R90"/>
@@
 <instance part="SUPPLY8" gate="GND" x="149.86" y="99.06" smashed="yes">
 <attribute name="VALUE" x="147.955" y="95.885" size="1.778" layer="96"/>
-</instance>
-<instance part="SUPPLY11" gate="G$1" x="86.36" y="78.74" smashed="yes" rot="R90">
-<attribute name="VALUE" x="83.185" y="76.835" size="1.778" layer="96" rot="R90"/>
 </instance>
 <instance part="BAT" gate="-2" x="116.84" y="101.6" smashed="yes">
@@
 <pinref part="C11" gate="G$1" pin="2"/>
 <pinref part="GND56" gate="GND" pin="GND"/>
-</segment>
-<segment>
-<pinref part="JP_5V" gate="A" pin="2"/>
-<pinref part="GND95" gate="GND" pin="GND"/>
-<wire x1="124.46" y1="73.66" x2="124.46" y2="76.2" width="0.1524" layer="91"/>
-<wire x1="124.46" y1="76.2" x2="127" y2="76.2" width="0.1524" layer="91"/>
-</segment>
-<segment>
-<pinref part="JP_9V" gate="A" pin="2"/>
-<wire x1="96.52" y1="76.2" x2="93.98" y2="76.2" width="0.1524" layer="91"/>
-<pinref part="GND96" gate="GND" pin="GND"/>
-<wire x1="93.98" y1="76.2" x2="93.98" y2="73.66" width="0.1524" layer="91"/>
 </segment>
 <segment>
@@
 <wire x1="193.04" y1="129.54" x2="193.04" y2="134.62" width="0.1524" layer="91"/>
 </segment>
-<segment>
-<pinref part="JP_5V" gate="A" pin="1"/>
-<pinref part="P+17" gate="1" pin="+5V"/>
-<wire x1="121.92" y1="78.74" x2="127" y2="78.74" width="0.1524" layer="91"/>
-</segment>
 </net>
 <net name="+9V" class="2">
 <segment>
-<pinref part="SUPPLY11" gate="G$1" pin="+9V"/>
-<pinref part="JP_9V" gate="A" pin="1"/>
-<wire x1="88.9" y1="78.74" x2="96.52" y2="78.74" width="0.1524" layer="91"/>
-</segment>
-<segment>
 <pinref part="C6" gate="G$1" pin="1"/>
