File: eagle_design_files/V4/mk312lite_V4.brd (EAGLE design)
At the start: 90 x 120 mm, 100 parts, among them Q1 IRFL024, Q2 IRFL024, Q3 BSP170PH6327, Q4 IRFL024, Q5 IRFL024, Q6 BSP170PH6327, Q7 MMBT3904, Q8 MMBT3904, U1 ATMEGA16A, U10 LM358D, U3 4066D, U8B LTC1661, Y1 8MHZ

Commit message: Add files via upload
Parts:
- Q1, Q2, Q4, Q5: value IRFL024 -> ZXMN4A06GTA
Changed lines of the file:
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@@
 <attribute name="VALUE" x="68.58" y="38.1" size="1.27" layer="27"/>
 </element>
-<element name="Q1" library="MK312parts" package="SOT223" package3d_urn="urn:adsk.eagle:package:29522/2" value="IRFL024" x="24.13" y="52.07" smashed="yes" rot="MR180">
+<element name="Q1" library="MK312parts" package="SOT223" package3d_urn="urn:adsk.eagle:package:29522/2" value="ZXMN4A06GTA" x="24.13" y="52.07" smashed="yes" rot="MR180">
 <attribute name="ALTERNATIVE" value="IRL100HS" x="24.13" y="52.07" size="1.778" layer="28" rot="MR180" display="off"/>
 <attribute name="ALTERNATIVE2" value="IRLL2705" x="24.13" y="52.07" size="1.778" layer="28" rot="MR180" display="off"/>
@@
 <attribute name="VALUE" x="21.9075" y="53.6575" size="0.8128" layer="28" ratio="10" rot="MR180"/>
 </element>
-<element name="Q4" library="MK312parts" package="SOT223" package3d_urn="urn:adsk.eagle:package:29522/2" value="IRFL024" x="54.61" y="52.07" smashed="yes" rot="MR180">
+<element name="Q4" library="MK312parts" package="SOT223" package3d_urn="urn:adsk.eagle:package:29522/2" value="ZXMN4A06GTA" x="54.61" y="52.07" smashed="yes" rot="MR180">
 <attribute name="NAME" x="53.4035" y="52.6415" size="1.016" layer="26" ratio="18" rot="MR180"/>
 <attribute name="POPULARITY" value="0" x="54.61" y="52.07" size="1.778" layer="28" rot="MR180" display="off"/>
 <attribute name="VALUE" x="52.3875" y="53.6575" size="0.8128" layer="28" ratio="10" rot="MR180"/>
 </element>
-<element name="Q5" library="MK312parts" package="SOT223" package3d_urn="urn:adsk.eagle:package:29522/2" value="IRFL024" x="74.93" y="52.07" smashed="yes" rot="MR180">
+<element name="Q5" library="MK312parts" package="SOT223" package3d_urn="urn:adsk.eagle:package:29522/2" value="ZXMN4A06GTA" x="74.93" y="52.07" smashed="yes" rot="MR180">
 <attribute name="NAME" x="74.1045" y="52.6415" size="1.016" layer="26" ratio="18" rot="MR180"/>
 <attribute name="POPULARITY" value="0" x="74.93" y="52.07" size="1.778" layer="28" rot="MR180" display="off"/>
@@
 <attribute name="VALUE" x="64.77" y="52.07" size="1.27" layer="28" rot="MR270" align="center"/>
 </element>
-<element name="Q2" library="MK312parts" package="SOT223" package3d_urn="urn:adsk.eagle:package:29522/2" value="IRFL024" x="44.45" y="52.07" smashed="yes" rot="MR180">
+<element name="Q2" library="MK312parts" package="SOT223" package3d_urn="urn:adsk.eagle:package:29522/2" value="ZXMN4A06GTA" x="44.45" y="52.07" smashed="yes" rot="MR180">
 <attribute name="ALTERNATIVE" value="IRL100HS" x="44.45" y="52.07" size="1.778" layer="28" rot="MR180" display="off"/>
 <attribute name="ALTERNATIVE2" value="IRLL2705" x="44.45" y="52.07" size="1.778" layer="28" rot="MR180" display="off"/>
