File: eagle_design_files/V4/mk312lite_V4.sch (EAGLE design)
At the start: 100 parts, among them Q1 IRFL024, Q2 IRFL024, Q3 BSP170PH6327, Q4 IRFL024, Q5 IRFL024, Q6 BSP170PH6327, Q7 MMBT3904, Q8 MMBT3904, U1 ATMEGA16A, U10 LM358D, U3 4066D, U8B LTC1661, Y1 8MHZ

Commit message: Add files via upload
Parts:
- Q1, Q2, Q4, Q5: value IRFL024 -> ZXMN4A06GTA
Changed lines of the file:
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@@
 <part name="R40" library="rcl" library_urn="urn:adsk.eagle:library:334" deviceset="R-EU_" device="R0805" package3d_urn="urn:adsk.eagle:package:23553/2" value="100K"/>
 <part name="GND6" library="supply2" deviceset="GND" device=""/>
-<part name="Q1" library="MK312parts" deviceset="N-HEXFET-2D_?-*" device="SOT232" package3d_urn="urn:adsk.eagle:package:29522/2" technology="IRLL2705" value="IRFL024">
+<part name="Q1" library="MK312parts" deviceset="N-HEXFET-2D_?-*" device="SOT232" package3d_urn="urn:adsk.eagle:package:29522/2" technology="IRLL2705" value="ZXMN4A06GTA">
 <attribute name="ALTERNATIVE" value="IRL100HS"/>
 <attribute name="ALTERNATIVE2" value="IRLL2705"/>
@@
 <part name="GND12" library="supply2" deviceset="GND" device=""/>
 <part name="R52" library="rcl" library_urn="urn:adsk.eagle:library:334" deviceset="R-EU_" device="R0805" package3d_urn="urn:adsk.eagle:package:23553/2" value="10K"/>
-<part name="Q4" library="MK312parts" deviceset="N-HEXFET-2D_?-*" device="SOT232" package3d_urn="urn:adsk.eagle:package:29522/2" technology="IRLL2705" value="IRFL024"/>
-<part name="Q5" library="MK312parts" deviceset="N-HEXFET-2D_?-*" device="SOT232" package3d_urn="urn:adsk.eagle:package:29522/2" technology="IRLL2705" value="IRFL024"/>
+<part name="Q4" library="MK312parts" deviceset="N-HEXFET-2D_?-*" device="SOT232" package3d_urn="urn:adsk.eagle:package:29522/2" technology="IRLL2705" value="ZXMN4A06GTA"/>
+<part name="Q5" library="MK312parts" deviceset="N-HEXFET-2D_?-*" device="SOT232" package3d_urn="urn:adsk.eagle:package:29522/2" technology="IRLL2705" value="ZXMN4A06GTA"/>
 <part name="R50" library="rcl" library_urn="urn:adsk.eagle:library:334" deviceset="R-EU_" device="R0805" package3d_urn="urn:adsk.eagle:package:23553/2" value="10K"/>
 <part name="C40" library="rcl" library_urn="urn:adsk.eagle:library:334" deviceset="C-EU" device="C0805" package3d_urn="urn:adsk.eagle:package:23617/2" value="0.1uF"/>
@@
 <part name="UART" library="jumper" library_urn="urn:adsk.eagle:library:252" deviceset="JP1E" device="" package3d_urn="urn:adsk.eagle:package:15455/1"/>
 <part name="Q6" library="SamacSys_Parts" deviceset="IRFL9014TRPBF" device="" value="BSP170PH6327"/>
-<part name="Q2" library="MK312parts" deviceset="N-HEXFET-2D_?-*" device="SOT232" package3d_urn="urn:adsk.eagle:package:29522/2" technology="IRLL2705" value="IRFL024">
+<part name="Q2" library="MK312parts" deviceset="N-HEXFET-2D_?-*" device="SOT232" package3d_urn="urn:adsk.eagle:package:29522/2" technology="IRLL2705" value="ZXMN4A06GTA">
 <attribute name="ALTERNATIVE" value="IRL100HS"/>
 <attribute name="ALTERNATIVE2" value="IRLL2705"/>
