File: eagle_design_files/V4/mk312lite_V4a.brd (EAGLE design)
At the start: 90 x 120 mm, 104 parts, among them IC1 LM2674, Q1 ZXMN4A06GTA, Q2 ZXMN4A06GTA, Q3 BSP170PH6327, Q4 ZXMN4A06GTA, Q5 ZXMN4A06GTA, Q6 BSP170PH6327, Q7 MMBT3904, Q8 MMBT3904, U1 ATMEGA16A, U10 LM358D, U3 4066D, U8B LTC1661, Y1 8MHZ

Commit message: Add files via upload
Parts:
- C9: value 100nF -> 10nF
- L1: value 68uH -> 47uH
Changed lines of the file:
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@@
 <attribute name="VALUE" x="40.95" y="6.39" size="1.27" layer="28" rot="MR90"/>
 </element>
-<element name="C9" library="rcl" library_urn="urn:adsk.eagle:library:334" package="C0805" package3d_urn="urn:adsk.eagle:package:23617/2" value="100nF" x="17.78" y="46.99" smashed="yes" rot="MR90">
+<element name="C9" library="rcl" library_urn="urn:adsk.eagle:library:334" package="C0805" package3d_urn="urn:adsk.eagle:package:23617/2" value="10nF" x="17.78" y="46.99" smashed="yes" rot="MR90">
 <attribute name="NAME" x="18.161" y="44.45" size="1.27" layer="26" rot="MR270"/>
 <attribute name="POPULARITY" value="88" x="3.81" y="69.85" size="1.778" layer="28" rot="MR90" display="off"/>
@@
 <attribute name="VALUE" x="13.335" y="41.91" size="0.4064" layer="28" rot="MR270"/>
 </element>
-<element name="L1" library="MK312parts" package="SMNR4030-151MT" package3d_urn="urn:adsk.eagle:package:14501/1" value="68uH" x="12.7" y="46.99" smashed="yes" rot="MR180">
+<element name="L1" library="MK312parts" package="SMNR4030-151MT" package3d_urn="urn:adsk.eagle:package:14501/1" value="47uH" x="12.7" y="46.99" smashed="yes" rot="MR180">
 <attribute name="NAME" x="11.844" y="47.61" size="1.27" layer="26" rot="MR180"/>
 <attribute name="POPULARITY" value="1" x="39.37" y="52.07" size="1.778" layer="28" rot="MR180" display="off"/>
