File: eagle_design_files/V4/mk312lite_V4a.sch (EAGLE design)
At the start: 104 parts, among them IC1 LM2674, Q1 ZXMN4A06GTA, Q2 ZXMN4A06GTA, Q3 BSP170PH6327, Q4 ZXMN4A06GTA, Q5 ZXMN4A06GTA, Q6 BSP170PH6327, Q7 MMBT3904, Q8 MMBT3904, U1 ATMEGA16A, U10 LM358D, U3 4066D, U8B LTC1661, Y1 8MHZ

Commit message: Add files via upload
Parts:
- C9: value 100nF -> 10nF
- L1: value 68uH -> 47uH
Changed lines of the file:
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@@
 <part name="F1" library="varistor" library_urn="urn:adsk.eagle:library:410" deviceset="VARISTOR" device="CN1812" package3d_urn="urn:adsk.eagle:package:30610/1" value="SMD1812P110TF"/>
 <part name="IC1" library="Eagle-JeeLabs" deviceset="LM2674" device=""/>
-<part name="L1" library="MK312parts" deviceset="SMNR4030-151MT" device="" package3d_urn="urn:adsk.eagle:package:14501/1" value="68uH"/>
+<part name="L1" library="MK312parts" deviceset="SMNR4030-151MT" device="" package3d_urn="urn:adsk.eagle:package:14501/1" value="47uH"/>
 <part name="D2" library="diode" library_urn="urn:adsk.eagle:library:210" deviceset="S1M" device="" package3d_urn="urn:adsk.eagle:package:43460/3" value="SS14"/>
 <part name="P+1" library="supply1" library_urn="urn:adsk.eagle:library:371" deviceset="+5V" device=""/>
-<part name="C9" library="rcl" library_urn="urn:adsk.eagle:library:334" deviceset="C-EU" device="C0805" package3d_urn="urn:adsk.eagle:package:23617/2" value="100nF"/>
+<part name="C9" library="rcl" library_urn="urn:adsk.eagle:library:334" deviceset="C-EU" device="C0805" package3d_urn="urn:adsk.eagle:package:23617/2" value="10nF"/>
 <part name="SUPPLY11" library="supply2" library_urn="urn:adsk.eagle:library:372" deviceset="GND" device=""/>
 <part name="SUPPLY15" library="supply1" library_urn="urn:adsk.eagle:library:371" deviceset="+12V" device=""/>
